File: backplane/kicad/a7s_backplane_routed.kicad_pcb (KiCad board)
At the start: 2 copper layers, 86.2 x 74.1 mm, 26 parts, among them J1 Conn_02x15_Odd_Even, J10 ENC, J11 BTN5_6, J12 FLIPPER, J2 Conn_01x15, J3 Conn_01x14, J5 Conn_02x04_Odd_Even, J5b Conn_01x01, J6 Conn_02x04_Odd_Even, J6b Conn_01x01, J8 JOY, SW1 SW_Push, SW2 SW_Push, SW3 SW_Push, SW4 SW_Push

Commit message: v2 silkscreens
Parts:
- added G***: DC34_JACK_W20, a7s:DC34_JACK_W20, F.Cu at (62.6, 43.8)
- added G***: AMNESIA_BRAIN_W12, a7s:AMNESIA_BRAIN_W12, B.Cu at (71.5, 78.5)
Other:
- board text added: "1.21GW"
- board text added: "DefCon34 CyberDeck by skitz0"
- board text added: "DefCon34 Cyberdeck Backplane v2 - skitz0@amnesia-labs.com"
- board text added: "FLIPPER GPIO: KBEMBEDDED/FLIPPER-GPIO-EDA"
- board text added: "HACK THE PLANET"
- board text added: "I don't care that they stole my idea's... I care that they don't have any of their own. - Nikola Tesla"
- board text added: "Special Thanks: @Hunny & @Buddah Maker Village @Nothingness and the full Goon Squad Hackers Guild PGH Amnesia-Labs.com"
- board text added: "What is right is not always popular, and what is popular is not always right. - Albert Einstein"
